File: pcb/BinaryVoltageIndicator.kicad_sch (KiCad schematic)
At the start: 11 parts, among them J1 Conn, Q1 2N7002, U1 MCP65R41-2402

Commit message: fix: change measurement resistors to 0603
the 0402 resistors in JLCPCBs standard library are 5% - too much for this to work properly
Parts:
- R1: footprint Resistor_SMD:R_0402_1005Metric -> Resistor_SMD:R_0603_1608Metric; LCSC C3017587 -> C22797
- R2: footprint Resistor_SMD:R_0402_1005Metric -> Resistor_SMD:R_0603_1608Metric; LCSC C25752 -> C22790
Changed lines of the file:
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@@
 			)
 		)
-		(property "Footprint" "Resistor_SMD:R_0402_1005Metric"
+		(property "Footprint" "Resistor_SMD:R_0603_1608Metric"
 			(at 92.71 90.17 0)
 			(effects
@@
 			)
 		)
-		(property "LCSC" "C25752"
+		(property "LCSC" "C22790"
 			(at 92.71 90.17 0)
 			(effects
@@
 			)
 		)
-		(property "Footprint" "Resistor_SMD:R_0402_1005Metric"
+		(property "Footprint" "Resistor_SMD:R_0603_1608Metric"
 			(at 92.71 80.01 0)
 			(effects
@@
 			)
 		)
-		(property "LCSC" "C3017587"
+		(property "LCSC" "C22797"
 			(at 92.71 80.01 0)
 			(effects
